File: Lecture Slides/Examples/Myduino/Myduino.brd (EAGLE design)
At the start: 160 x 100 mm, 30 parts, among them J2 GENERIC-BATTERY-CONN-RECEPTAC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, SW1 PUSHBUTTON-SHIELD-GND_CK_KMR2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, U1 ATMEGA328-NO-THERMAL_32TQFP, U3 ADJUSTABLE-VOLTAGE-REGULATOR_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, Y1 16MHz

Commit message: new slides
Parts:
- moved Y1 117.5 mm to (-59.7, 43.2)
- moved JP3 109.3 mm to (-52.1, 58.4)
- moved D5 102.6 mm to (-20.3, 53.3)
- moved U1 95.4 mm to (-43.2, 17.8)
- moved R2 93.6 mm to (22.9, 86.4), turned to 90 degrees
- moved SW1 91.1 mm to (-69.8, 48.3)
- moved JP4 79.0 mm to (-52.1, 63.5)
- moved R5 78.8 mm to (-17.8, 78.7)
- moved R2C2 74.1 mm to (14.0, 91.4)
- moved D4 72.7 mm to (-43.2, 43.2)
- moved J2 65.0 mm to (-58.4, 27.9), turned to 0 degrees
- moved SET_VOLTAGE1 57.5 mm to (11.4, 95.2)
- moved D3 56.0 mm to (-22.9, 43.2)
- moved JP1 55.8 mm to (-48.3, 6.35), turned to 0 degrees
- moved C6 52.3 mm to (7.62, 85.1), turned to 90 degrees
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